File: CavityDentureForM5Stack.kicad_pcb (KiCad board)
At the start: 2 copper layers, 54 x 54 mm, 13 parts, among them J1 free_holes

Commit message: Correct label for 35 pin
Other:
- board text added: "35/AD"
Changed lines of the file:
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@@
-(kicad_pcb (version 20171130) (host pcbnew 5.1.4-e60b266~84~ubuntu18.04.1)
+(kicad_pcb (version 20171130) (host pcbnew 5.1.5-52549c5~86~ubuntu18.04.1)
   (general
     (thickness 1.6)
@@
     (effects (font (size 0.7 0.7) (thickness 0.175)))
   )
-  (gr_text 36/AD (at 132.0488 56.6232) (layer F.SilkS)
-    (effects (font (size 0.7 0.7) (thickness 0.175)))
-  )
+  (gr_text 35/AD (at 132.0488 56.6232) (layer F.SilkS)
+    (effects (font (size 0.7 0.7) (thickness 0.175)))
+  )
